Commit message: 2

File: src/racecar_description/urdf/sensors/camera.xacro (robot description, xacro)
@@ -2,63 +2,61 @@
 <robot xmlns:xacro="http://www.ros.org/wiki/xacro" name="camera">
 	<link name="camera_link">
-	    <inertial>
-		<mass value="0.001" />
-		<origin xyz="0 0 0" />
-		<inertia ixx="0.001" ixy="0.0" ixz="0.0"
-		         iyy="0.001" iyz="0.0"
-		         izz="0.001" />
-	    </inertial>
-	    <visual>
-		<origin xyz=" 0 0 0 " rpy="1.57 0 1.57" />
-		<geometry>
-		    <mesh filename="package://racecar_description/meshes/S1030-0315.dae" scale="0.1 0.1 0.1" />
-		</geometry>
-	    </visual>
-	    <collision>
-		<origin xyz="0.0 0.0 0.0" rpy="0 0 0" />
-		<geometry>
-		    <box size="0.03 0.16 0.03" />
-		</geometry>
-	    </collision>
+		<inertial>
+			<mass value="0.001" />
+			<origin xyz="0 0 0" />
+			<inertia ixx="0.001" ixy="0.0" ixz="0.0" iyy="0.001" iyz="0.0" izz="0.001" />
+		</inertial>
+		<visual>
+			<origin xyz=" 0 0 0 " rpy="1.57 0 1.57" />
+			<geometry>
+				<mesh filename="package://racecar_description/meshes/S1030-0315.dae" scale="0.1 0.1 0.1" />
+			</geometry>
+		</visual>
+		<collision>
+			<origin xyz="0.0 0.0 0.0" rpy="0 0 0" />
+			<geometry>
+				<box size="0.03 0.16 0.03" />
+			</geometry>
+		</collision>
 	</link>
 	<gazebo reference="camera_link">
-	<material>Gazebo/Black</material>
+		<material>Gazebo/Black</material>
 	</gazebo>
 	<gazebo reference="camera_link">
 		<sensor type="camera" name="camera_node">
 			<pose>0 0 0 0 0 0</pose>
-		        <update_rate>30.0</update_rate>
-		        <camera name="head">
-		            <horizontal_fov>1.3962634</horizontal_fov>
-		            <image>
-		                <width>1280</width>
-		                <height>720</height>
-		                <format>R8G8B8</format>
-		            </image>
-		            <clip>
-		                <near>0.02</near>
-		                <far>300</far>
-		            </clip>
-		            <noise>
-		                <type>gaussian</type>
-		                <mean>0.0</mean>
-		                <stddev>0.007</stddev>
-		            </noise>
-		        </camera>
-		        <plugin name="gazebo_camera" filename="libgazebo_ros_camera.so">
-		            <alwaysOn>true</alwaysOn>
-		            <updateRate>0.0</updateRate>
-		            <cameraName>/camera</cameraName>
-		            <imageTopicName>image_raw</imageTopicName>
-		            <cameraInfoTopicName>camera_info</cameraInfoTopicName>
-		            <frameName>camera_link</frameName>
-		            <hackBaseline>0.07</hackBaseline>
-		            <distortionK1>0.0</distortionK1>
-		            <distortionK2>0.0</distortionK2>
-		            <distortionK3>0.0</distortionK3>
-		            <distortionT1>0.0</distortionT1>
-		            <distortionT2>0.0</distortionT2>
-		        </plugin>
-		    </sensor>
-	  </gazebo>
+			<update_rate>30.0</update_rate>
+			<camera name="head">
+				<horizontal_fov>1.3962634</horizontal_fov>
+				<image>
+					<width>1280</width>
+					<height>720</height>
+					<format>R8G8B8</format>
+				</image>
+				<clip>
+					<near>0.02</near>
+					<far>300</far>
+				</clip>
+				<noise>
+					<type>gaussian</type>
+					<mean>0.0</mean>
+					<stddev>0.007</stddev>
+				</noise>
+			</camera>
+			<plugin name="gazebo_camera" filename="libgazebo_ros_camera.so">
+				<alwaysOn>true</alwaysOn>
+				<updateRate>0.0</updateRate>
+				<cameraName>/camera</cameraName>
+				<imageTopicName>image_raw</imageTopicName>
+				<cameraInfoTopicName>camera_info</cameraInfoTopicName>
+				<frameName>camera_link</frameName>
+				<hackBaseline>0.07</hackBaseline>
+				<distortionK1>0.0</distortionK1>
+				<distortionK2>0.0</distortionK2>
+				<distortionK3>0.0</distortionK3>
+				<distortionT1>0.0</distortionT1>
+				<distortionT2>0.0</distortionT2>
+			</plugin>
+		</sensor>
+	</gazebo>
 </robot>

File: src/racecar_description/urdf/sensors/imu.xacro (robot description, xacro)
@@ -7,7 +7,5 @@
                 <mass value="0.001" />
                 <origin xyz="0 0 0" />
-                <inertia ixx="0.001" ixy="0.0" ixz="0.0"
-                         iyy="0.001" iyz="0.0"
-                         izz="0.001" />
+                <inertia ixx="0.001" ixy="0.0" ixz="0.0" iyy="0.001" iyz="0.0" izz="0.001" />
             </inertial>
             <visual>

File: src/racecar_description/urdf/sensors/lidar.xacro (robot description, xacro)
@@ -7,7 +7,5 @@
                 <mass value="0.001" />
                 <origin xyz="0 0 0" />
-                <inertia ixx="0.001" ixy="0.0" ixz="0.0"
-                         iyy="0.001" iyz="0.0"
-                         izz="0.001" />
+                <inertia ixx="0.001" ixy="0.0" ixz="0.0" iyy="0.001" iyz="0.0" izz="0.001" />
             </inertial>
             <visual>
